File: Eagle/RFBoardV3/main.brd (EAGLE design)
At the start: 34.3 x 77.5 mm, 25 parts, among them Q1 8/16/20MHz, U1 ATMEGA328

Commit message: Changed reed/term to OR instead of AND
Connections:
- net D5: no longer S3.1
- net SCREW_TERM: now also S3.1
Routing:
- net SCREW_TERM: track 10.2 -> 13.7 mm
- net D5: track 66.8 -> 68.5 mm
Changed lines of the file:
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@@
 <?xml version="1.0" encoding="utf-8"?>
 <!DOCTYPE eagle SYSTEM "eagle.dtd">
-<eagle version="7.2.0">
+<eagle version="7.1.0">
 <drawing>
 <settings>
@@
 <wire x1="28.194" y1="73.6092" x2="26.8224" y2="72.2376" width="0.1524" layer="1"/>
 <wire x1="28.194" y1="73.6092" x2="28.25" y2="73.66" width="0.1524" layer="1"/>
+<contactref element="S3" pad="1"/>
+<wire x1="28.575" y1="64.77" x2="32.0675" y2="64.77" width="0.1524" layer="1"/>
 </signal>
 <signal name="D5">
 <contactref element="U1" pad="9"/>
 <contactref element="JP2" pad="1"/>
-<contactref element="S3" pad="1"/>
 <wire x1="28.0416" y1="15.6972" x2="23.5458" y2="11.2014" width="0.1524" layer="1"/>
 <wire x1="28.0416" y1="23.4696" x2="28.0416" y2="15.6972" width="0.1524" layer="16"/>
 <wire x1="32.8422" y1="28.2702" x2="28.0416" y2="23.4696" width="0.1524" layer="16"/>
 <wire x1="32.8422" y1="64.008" x2="32.8422" y2="28.2702" width="0.1524" layer="16"/>
-<wire x1="32.0802" y1="64.77" x2="32.8422" y2="64.008" width="0.1524" layer="16"/>
 <wire x1="23.5458" y1="11.2014" x2="23.505940625" y2="11.2013375" width="0.1524" layer="1"/>
-<wire x1="32.0802" y1="64.77" x2="32.0675" y2="64.77" width="0.1524" layer="16"/>
-<wire x1="31.7754" y1="64.9986" x2="31.7754" y2="73.6092" width="0.1524" layer="1"/>
-<wire x1="32.004" y1="64.77" x2="31.7754" y2="64.9986" width="0.1524" layer="1"/>
 <wire x1="31.7754" y1="73.6092" x2="31.75" y2="73.66" width="0.1524" layer="1"/>
-<wire x1="32.004" y1="64.77" x2="32.0675" y2="64.77" width="0.1524" layer="1"/>
 <via x="28.0416" y="15.6972" extent="1-16" drill="0.3302"/>
+<wire x1="32.8422" y1="64.008" x2="33.3375" y2="64.008" width="0.1524" layer="16"/>
+<wire x1="33.3375" y1="64.008" x2="33.3375" y2="73.66" width="0.1524" layer="16"/>
+<wire x1="33.3375" y1="73.66" x2="31.75" y2="73.66" width="0.1524" layer="16"/>
 </signal>
 <signal name="N$4">
