File: Eagle/RFBoardV4/main.brd (EAGLE design)
At the start: 34.3 x 77.5 mm, 32 parts, among them Q1 8/16/20MHz, U1 ATMEGA328

Commit message: Added TDK inductor
Parts:
- removed C6: 4.7uH, SparkFun:0805
- added L1: VLF302510MT, inductor-tdk:VLF302510MT
Changed lines of the file:
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@@
 <element name="C4" library="SparkFun" package="0603-CAP" value="10uF" x="-6.6675" y="-5.08"/>
 <element name="C5" library="SparkFun" package="0603-CAP" value="4.7uF" x="-6.6675" y="-8.255"/>
-<element name="C6" library="SparkFun" package="0805" value="4.7uH" x="-9.8425" y="-7.9375"/>
+<element name="L1" library="inductor-tdk" package="VLF302510MT" value="VLF302510MT" x="-14.9225" y="-6.985"/>
 </elements>
 <signals>
